File: nRF9151_power_rf.kicad_sch (KiCad schematic)
At the start: 25 parts, among them J1 CONMHF1-SMD-G-T, U1 nRF9151-LACA, U2 SKY65943-11

Commit message: Add files via upload
Other:
- title: Low Power LTE & GNSS SiP -> nRF9151 - Low Power LTE & GNSS SiP
Changed lines of the file:
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@@
 	(paper "A4")
 	(title_block
-		(title "Low Power LTE & GNSS SiP")
+		(title "nRF9151 - Low Power LTE & GNSS SiP")
 		(date "2025-01-04")
 		(rev "A")

Commit message: Publish PCB and Schematics
Parts:
- C1: value 0.1u 16V -> 100n 16V; Category Capacitors -> Capacitors/Ceramic Capacitors
- C10: renamed from C11; Part-DB Footprint (none) -> 0201; Part-DB ID 36 -> 109
- C11: renamed from C10; Part-DB Footprint (none) -> 0201; Part-DB ID 36 -> 109
- C12: renamed from C9; value 0.1u 16V -> 100n 16V; Category Capacitors -> Capacitors/Ceramic Capacitors
- C4: renamed from C5; value 0.1u 16V -> 100n 16V; Category Capacitors -> Capacitors/Ceramic Capacitors
- C6: renamed from C7; value 4.7u 10V -> 4u7 10V
- C7: renamed from C6; value 0.1u 16V -> 100n 16V; Category Capacitors -> Capacitors/Ceramic Capacitors
- C8: value 4.7u 10V -> 4u7 10V
- C9: renamed from C12; value 0.1u 16V -> 100n 16V; Category Capacitors -> Capacitors/Ceramic Capacitors
- J11: renamed from J1; footprint footprints:CONMHF1-SMD -> footprints:TE_CONN_MHF1_SMD; now in the parts list
- L2: value 9.1n -> 9n1
- R4: renamed from R3; footprint footprints:R_0402_1005Metric -> footprints:R_0201_0603Metric; symbol DB:ERJ-2GE0R00X -> DB:ERJ-1GN0R00C; MPN ERJ-2GE0R00X -> ERJ-1GN0R00C; Part-DB Footprint 0402 -> 0201; Part-DB ID 19 -> 134
- R5: renamed from R6; footprint footprints:R_0402_1005Metric -> footprints:R_0201_0603Metric; symbol DB:ERJ-2GE0R00X -> DB:ERJ-1GN0R00C; MPN ERJ-2GE0R00X -> ERJ-1GN0R00C; Part-DB Footprint 0402 -> 0201; Part-DB ID 19 -> 134
- R6: renamed from R7; footprint footprints:R_0402_1005Metric -> footprints:R_0201_0603Metric; symbol DB:ERJ-2GE0R00X -> DB:ERJ-1GN0R00C; MPN ERJ-2GE0R00X -> ERJ-1GN0R00C; Part-DB Footprint 0402 -> 0201; Part-DB ID 19 -> 134
- U1: footprint footprints:nRF9151-LACA -> footprints:NORDIC_LGA-113
- U2: footprint footprints:SKY65943-11 -> footprints:SKY_MCM-10
- renumbered C4 to C5, R8 to R3, R5 to R7, R4 to R8
