File: nrf9151_gpio_uicc.kicad_sch (KiCad schematic)
At the start: 17 parts, among them J2 SF72S006VBDR2500, J6 BD125-10-A-0305-0580-L-B, U1 nRF9151-LACA, U3 MX25V8035FZUI, U4 EMIF03-SIM02M8

Commit message: Add files via upload
Other:
- title: (none) -> nRF9151 - GPIO + UICC
Changed lines of the file:
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@@
 	(paper "A4")
 	(title_block
+		(title "nRF9151 - GPIO + UICC")
 		(date "2025-01-04")
 	)

Commit message: Publish PCB and Schematics
Parts:
- removed J6: BD125-10-A-0305-0580-L-B, footprints:BD125-10-A-0305-0580-L-B, symbol DB:BD125-10-A-0305-0580-L-B
- added J12: FTSH-105-01-L-DV-K, footprints:SAM_MICRO-IDC_FTSH-105-01-L-DV-K_SMD, symbol DB:FTSH-105-01-L-DV-K
- added R24: 10K, footprints:R_0402_1005Metric, symbol DB:ERJ-2RKF1002X
- added R25, R36, R37: 590, footprints:R_0402_1005Metric, symbol db:ERJ-2RKF5900X
- added SW1: PTS636SM50JSMTR LFS, footprints:SW_Tactile_SPST_NO_Straight_CK_ PTS636SM50JSMTR LFS, symbol DB:PTS636SM50JSMTR LFS
- C13: renamed from C14; Part-DB Footprint (none) -> 0402
- C14: renamed from C13; value 0.1u 16V -> 100n 16V; Category Capacitors -> Capacitors/Ceramic Capacitors
- C15: value 0.1u 16V -> 100n 16V; Category Capacitors -> Capacitors/Ceramic Capacitors
- J13: renamed from J2; footprint footprints:SF72S006VBDR2500 -> footprints:JAE_SF72S006VBDR2500
- U1: footprint footprints:nRF9151-LACA -> footprints:NORDIC_LGA-113
- U3: renamed from U4; footprint footprints:EMIF03-SIM02M8 -> footprints:ST_UFDFN-8
- renumbered R9 to R10, R10 to R11, R11 to R12, R12 to R13, R13 to R14, R23 to R9, U3 to U4
Connections:
- net I2C_PMIC_SCL is gone; now on net I2C_PMIC.SCL: R10.2
- net I2C_PMIC_SDA is gone; now on net I2C_PMIC.SDA: R12.2
- net nQON is gone; now on net nCE: U1.80 (P0.19)
- net APP_SIM_DETECT: now also U1.12 (P0.25); no longer U1.50 (P0.31)
- net BOOST_PWM_EN: now also U1.11 (P0.24); no longer U1.6 (P0.22)
- net GND: now also U3.GND, U4.GND, J12.3 (GND), J12.5 (GND), J12.9 (GND), SW1.2
- net LED_GREEN: now also R37.2; no longer D1.1 (K)
- net LED_RED: now also R36.2; no longer D2.1 (K)
- net LED_YELLOW: now also U1.63 (P0.06), R25.2; no longer D3.1 (K), U1.68 (P0.09)
- net PANEL_DETECT: now also U1.79 (P0.18); no longer U1.49 (P0.30)
- net PWR_3V3H: now also J12.1 (VREF), R24.1
- net SPI_FLASH_SIO1: now also U1.57 (P0.01); no longer U1.59 (P0.03)
- net SPI_FLASH_SI/SIO0: now also U1.62 (P0.05); no longer U1.58 (P0.02)
- net SPI_FLASH_nHOLD/SIO3: now also U1.59 (P0.03); no longer U1.62 (P0.05)
- net SPI_FLASH_nWP/SIO2: now also U1.58 (P0.02); no longer U1.61 (P0.04)
- net nCE: no longer U1.79 (P0.18)
- net nINT: now also U1.6 (P0.22), R24.2; no longer U1.78 (P0.17)
- net I2C_PMIC.SCL: now reaches U1.2 (P0.20)
- net nRF_GPIO2: now reaches U1.44 (P0.26)
- net nRF_GPIO1: now reaches U1.45 (P0.27)
- net nRF_GPIO0: now reaches U1.47 (P0.28)
- net BLE_SPI.nCS: now reaches U1.48 (P0.29)
- net I2C_PMIC.SDA: now reaches U1.5 (P0.21)
- net BLE_SPI.MISO: now reaches U1.69 (P0.10)
- net BLE_SPI.MOSI: now reaches U1.70 (P0.11)
- net UART1.RX: now reaches U1.72 (P0.12)
- net UART1.TX: now reaches U1.73 (P0.13)
- net UART0.RX: now reaches U1.74 (P0.14)
- net UART0.TX: now reaches U1.75 (P0.15)
- net I2C_SBUS_SCL renamed I2C_SBUS.SCL
- net I2C_SBUS.SCL: now also U1.50 (P0.31)
- net I2C_SBUS_SDA renamed I2C_SBUS.SDA
- net I2C_SBUS.SDA: now also U1.49 (P0.30)
- net SPI_FLASH_SCLK_TERM renamed SCLK_TERM
- net SCLK_TERM: now also U1.61 (P0.04); no longer U1.57 (P0.01)
- net STAT renamed nRF52_nRESET
- net SWDCLK renamed nRF91_SWD.CLK
- net nRF91_SWD.CLK: now also J12.4 (SWDCLK)
- net SWDIO renamed nRF91_SWD.IO
- net nRF91_SWD.IO: now also J12.2 (SWDIO)
- net nRESET renamed nRF91_SWD.nRESET
- net nRF91_SWD.nRESET: now also J12.10 (nRST), SW1.1
- new net: D3.1 (K), R25.1
- new net: D1.1 (K), R37.1
- new net: D2.1 (K), R36.1
- new net BLE_SPI.CLK: U1.68 (P0.09)
- new net SWO_UNUSED: J12.6 (SWO)
- new net nRF91_SWD.SWO: U1.78 (P0.17)
- no-connect marks 28 -> 13
Other:
- moved on the sheet: C14, D1, D2, D3, R10, R11, R12, R13, R9, U1B, U4
