File: power_management.kicad_sch (KiCad schematic)
At the start: 50 parts, among them Q1 DMN1019UFDE-7, Q2 DMN1019UFDE-7, Q3 DMN1019UFDE-7, Q4 DMN1019UFDE-7, Q5 SSM3J355R,LF, U10 TPS22995RZFR, U6 BQ25798, U7 TPS631010YBGR

Commit message: Add files via upload
Other:
- title: (none) -> Power Management

Commit message: Publish PCB and Schematics
Parts:
- removed C21, C22, C25, C33, C34: 100n 50V, footprints:C_0603_1608Metric, symbol DB:CC0603KRX7R9BB104
- removed C45: 10u 10V, footprints:C0805C106K8PACTU, symbol DB:C0805C106K8PACTU
- removed L5: 1u, footprints:74404043010A, symbol DB:74404043010A
- removed Q5: SSM3J355R,LF, footprints:TOSHIBA_SOT-23F, symbol DB:SSM3J355R,LF
- removed R25, R28, R29, R30: 10K, footprints:R_0402_1005Metric, symbol DB:ERJ-2RKF1002X
- removed R32: 100k, footprints:R_0402_1005Metric, symbol DB:RC0402FR-07100KL
- removed R33: 360k, footprints:R_0402_1005Metric, symbol DB:RC0402FR-07360KL
- added C19, C20, C23, C24, C32: 100n 50V, footprints:C_0402_1005Metric, symbol DB:GRM155R71H104KE14D
- added C28: 10u 10V, footprints:C_0805_2012Metric, symbol DB:C0805C106K8PACTU
- added C59, C60: 10u 25V, footprints:C_0805_2012Metric, symbol DB:GRM21BR61E106KA73L
- added J14: 10129380-902001BLF, footprints:PinHeader_1x02_P2.54mm_Vertical_SMD_Pin1Left, symbol DB:10129380-902001BLF
- added JMP7: QPC02SXGN-RC, symbol DB:QPC02SXGN-RC
- added L4: 1u, footprints:L_Taiyo-Yuden_MD-3030, symbol DB:LSXND3030QKT1R0NNG
- added R18, R22, R23: 10K, footprints:R_0402_1005Metric, symbol DB:ERJ-2RKF1002X
- added R26: 215k, footprints:R_0402_1005Metric, symbol DB:RC0402FR-07215KL
- added R27: 59k, footprints:R_0402_1005Metric, symbol DB:RC0402FR-0759KL
- added TP8: TestPoint_Small, footprints:TestPoint_Pad_1.0x1.0mm, symbol DB:Test Point, Small
- L3: renamed from L4; value 1u0 -> 1u
- Q1, Q4: footprint footprints:DI_DFN2020 -> footprints:DI_DFN2020-6
- Q2: renamed from Q3; footprint footprints:DI_DFN2020 -> footprints:DI_DFN2020-6
- Q3: renamed from Q2; footprint footprints:DI_DFN2020 -> footprints:DI_DFN2020-6
- R16: renamed from R18; footprint symbols:R_0402_1005Metric -> footprints:R_0402_1005Metric
- R17: renamed from R19; footprint symbols:R_0402_1005Metric -> footprints:R_0402_1005Metric
- R28: renamed from R24; value 30.1k -> 30k1; footprint footprints: R_0402_1005Metric -> footprints:R_0402_1005Metric
- R29: renamed from R31; value 5.23k -> 5k23; footprint footprints: R_0402_1005Metric -> footprints:R_0402_1005Metric
- U5: renamed from U6; footprint footprints:TI_QFN-29 -> footprints:TI_VQFN-HR-29
- U6: renamed from U7; footprint footprints:TPS631010YBGR -> footprints:TI_DSBGA-8
- U7: renamed from U10; footprint footprints:TPS22995RZFR -> footprints:TI_WQFN-6
- renumbered C23 to C16, C19 to C17, C24 to C18, C20 to C21, C32 to C22, C17 to C25, C18 to C26, C31 to C27, C41 to C29, C35 to C30, C47 to C31, C36 to C33, C37 to C34, C43 to C35, C38 to C36, C46 to C37, C39 to C38, C40 to C39, C44 to C40, R20 to R15, R22 to R19, R26 to R20, R27 to R21, R35 to R30
Connections:
- net BAT is gone; now on net PWR_BATT: R19.2, U5.22 (BAT), U5.23 (BAT)
- net BOOST_PWM_EN: now also R18.1; no longer U7.3 (ON)
- net GND: now also C19.2, C20.2, C23.2, C24.2, C28.2, C32.2, C59.2, C60.2, R18.2, R27.2; no longer C31.2
- net ILIM_HIZ: now also R26.2, R27.1
- net PMID: now also C24.1
- net PWR_3V3: now also R22.1, R23.1
- net PWR_BATT: now also C31.2, C59.1, C60.1
- net PWR_SOLAR: now also Q2.1 (D), C19.1; no longer Q2.3 (D)
- net PWR_USB_5V0: now also Q1.1 (D), C20.1; no longer Q1.3 (D)
- net PWR_VBUS: now also Q3.1 (D), Q4.1 (D), C23.1; no longer Q3.3 (D), Q4.3 (D)
- net REGN: now also R26.1
- net SBUS_EN: now also U7.3 (ON)
- net STAT: now also R23.2, TP8.1
- net nCE: now also R22.2
- net ACDRV2_G: now reaches C26.1, R17.1
- net ACDRV2_G: now also Q2.3 (G), Q4.3 (G); no longer Q2.2 (G), Q4.2 (G)
- net CT: now reaches C40.2, U7.6 (CT)
- net at U6.B1 (LX1): now also L4.1
- net at U6.C1 (LX2): now also L4.2
- net FB: now reaches R20.2, R21.1, U6.D2 (FB)
- net ACDRV1_G: now reaches C25.2, R16.1
- net ACDRV1_G: now also Q1.3 (G), Q3.3 (G); no longer Q1.2 (G), Q3.2 (G)
- net BTST2: now reaches C30.1, U5.19 (BTST2)
- net SW2: now reaches C30.2, L3.2, U5.26 (SW2)
- net SW1: now reaches C29.2, L3.1, U5.28 (SW1)
- net BTST1: now reaches C29.1, U5.4 (BTST1)
- net I2C_PMIC_SCL renamed I2C_PMIC.SCL
- net I2C_PMIC_SDA renamed I2C_PMIC.SDA
- net SYS renamed PWR_SYS
- net PWR_SYS: now also C32.1, J14.2 (Pin_2); no longer U6.A1 (VIN), U6.A2 (EN)
- new net ACDRV1_S: C25.1, Q1.4 (S), Q3.4 (S)
- new net ACDRV2_S: C26.2, Q2.4 (S), Q4.4 (S)
- new net PWR_TPS63_VIN: C28.1, J14.1 (Pin_1), U6.A1 (VIN), U6.A2 (EN)
- no-connect marks 2 -> 3
Other:
- moved on the sheet: C29, C30, C31, C37, L3
