File: solar-ribbit.kicad_sch (KiCad schematic)
At the start: 4 parts, among them CN1 SM04B-SRSS-TB, J3 3.5mm/1.1mm, J4 AA-CONTACT-SMD, J5 AA-CONTACT-SMD

Commit message: Add files via upload
Parts:
- removed CN1: SM04B-SRSS-TB, footprints:JST_SH_SM04B-SRSS-TB, symbol DB:SM04B-SRSS-TB
- added J7: BM04B-SRSS-TB, footprints:BM04B-SRSS-TB, symbol DB:BM04B-SRSS-TB
Connections:
- net GND: now also J7.1, J7.G1, J7.G2
- net I2C_SBUS_SCL: now also J7.4
- net I2C_SBUS_SDA: now also J7.3
- net Power Management/PWR_3V3_LS: now also J7.2
Other:
- note added: "3.5mm OD / 1.1mm ID Female DC Barrel Jack Connector"
- note added: "Pair of SMD contacts form a 14430 cell holder"
- note added: "to Sensor Bus"
- note added: "via STEMMA QT / QWIIC connector"
- note removed: "(Pair of SMD contacts form 14430 cell holder)"
- note removed: "Sensor Bus"
- title: (none) -> Solar Powered Ribbit Network Frog Sensor
Changed lines of the file:
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@@
 	(paper "A4")
 	(title_block
+		(title "Solar Powered Ribbit Network Frog Sensor")
 		(date "2025-01-04")
 	)
@@
 		)
 	)
+	(bus
+		(pts
+			(xy 182.88 58.42) (xy 195.58 58.42)
+		)
+		(stroke
+			(width 0)
+			(type default)
+		)
+	)
 	(wire
 		(pts
@@
 	(wire
 		(pts
-			(xy 233.68 109.22) (xy 247.65 109.22)
+			(xy 233.68 109.22) (xy 248.92 109.22)
 		)
 		(stroke
@@
 	(wire
 		(pts
-			(xy 191.77 77.47) (xy 199.39 77.47)
+			(xy 191.77 77.47) (xy 200.66 77.47)
 		)
 		(stroke
@@
 	(bus
 		(pts
-			(xy 196.85 57.15) (xy 184.15 57.15)
+			(xy 196.85 55.88) (xy 196.85 57.15)
 		)
 		(stroke
@@
 	(bus
 		(pts
-			(xy 196.85 55.88) (xy 196.85 57.15)
+			(xy 196.85 57.15) (xy 195.58 58.42)
 		)
 		(stroke
@@
 	(wire
 		(pts
-			(xy 240.03 77.47) (xy 232.41 77.47)
+			(xy 240.03 77.47) (xy 233.68 77.47)
 		)
 		(stroke
@@
 		)
 	)
-	(text "(Pair of SMD contacts form 14430 cell holder)"
+	(text "Pair of SMD contacts form\na 14430 cell holder"
 		(exclude_from_sim no)
-		(at 40.894 59.944 0)
+		(at 37.846 59.944 0)
 		(effects
 			(font
@@
 	(text "Battery Holder\n"
 		(exclude_from_sim no)
-		(at 41.148 55.372 0)
+		(at 38.1 54.864 0)
 		(effects
 			(font
@@
 		)
 	)
+	(text "via STEMMA QT / QWIIC\nconnector"
+		(exclude_from_sim no)
+		(at 258.318 52.832 0)
+		(effects
+			(font
+				(size 1.27 1.27)
+			)
+		)
+	)
 	(text "Solar Connector"
 		(exclude_from_sim no)
-		(at 42.672 94.996 0)
+		(at 39.37 92.71 0)
 		(effects
 			(font
@@
 		)
 	)
-	(text "Sensor Bus"
+	(text "to Sensor Bus"
 		(exclude_from_sim no)
-		(at 224.79 33.02 0)
+		(at 258.826 47.498 0)
 		(effects
 			(font
@@
 		)
 	)
+	(text "3.5mm OD / 1.1mm ID Female \nDC Barrel Jack Connector"
+		(exclude_from_sim no)
+		(at 38.862 98.044 0)
+		(effects
+			(font
+				(size 1.27 1.27)
+			)
+		)
+	)
 	(text "USB-C Connector\n"
 		(exclude_from_sim no)
-		(at 43.688 128.016 0)
+		(at 40.64 127.508 0)
 		(effects
 			(font
@@
 	)
 	(label "I2C_SBUS"
-		(at 184.15 57.15 0)
+		(at 182.88 58.42 0)
 		(fields_autoplaced yes)
 		(effects
@@
 	)
 	(label "PANEL_DETECT"
-		(at 247.65 109.22 180)
+		(at 248.92 109.22 180)
 		(fields_autoplaced yes)
 		(effects
@@
 				(path "/9ed354c1-be1e-4ed3-9daf-708fd38c762e"
 					(reference "J5")
+					(unit 1)
+				)
+			)
+		)
+	)
+	(symbol
+		(lib_id "DB:BM04B-SRSS-TB")
+		(at 223.52 50.8 0)
+		(unit 1)
+		(exclude_from_sim yes)
+		(in_bom yes)
+		(on_board yes)
+		(dnp no)
+		(fields_autoplaced yes)
+		(property "Reference" "J7"
+			(at 224.79 38.1 0)
+			(effects
+				(font
+					(size 1.27 1.27)
+				)
+			)
+		)
+		(property "Value" "BM04B-SRSS-TB"
+			(at 224.79 40.64 0)
+			(effects
+				(font
+					(size 1.27 1.27)
+				)
+			)
+		)
+		(property "Footprint" "footprints:BM04B-SRSS-TB"
+			(at 223.52 50.8 0)
+			(effects
+				(font
+					(size 1.27 1.27)
+				)
+				(hide yes)
+			)
+		)
+		(property "Datasheet" "http://parts.djgood.ca/en/part/102/info"
+			(at 223.52 50.8 0)
+			(effects
+				(font
+					(size 1.27 1.27)
+				)
+				(hide yes)
+			)
+		)
+		(property "Description" "Connector Header Surface Mount 4 position 0.039\" (1.00mm)"
+			(at 223.52 50.8 0)
+			(effects
+				(font
+					(size 1.27 1.27)
+				)
+				(hide yes)
+			)
+		)
+		(property "Category" "Connectors/Rectangular Connectors/Male Pins"
+			(at 223.52 50.8 0)
+			(effects
+				(font
+					(size 1.27 1.27)
+				)
+				(hide yes)
+			)
+		)
+		(property "MPN" "BM04B-SRSS-TB"
+			(at 223.52 50.8 0)
+			(effects
+				(font
+					(size 1.27 1.27)
+				)
+				(hide yes)
+			)
+		)
+		(property "Manufacturer" "JST Sales America Inc."
+			(at 223.52 50.8 0)
+			(effects
+				(font
+					(size 1.27 1.27)
+				)
+				(hide yes)
+			)
+		)
+		(property "Manufacturing Status" "Active"
+			(at 223.52 50.8 0)
+			(effects
+				(font
+					(size 1.27 1.27)
+				)
+				(hide yes)
+			)
+		)
+		(property "Part-DB ID" "102"
+			(at 223.52 50.8 0)
+			(effects
+				(font
+					(size 1.27 1.27)
+				)
+				(hide yes)
+			)
+		)
+		(pin "G2"
+		)
+		(pin "1"
+		)
+		(pin "4"
+		)
+		(pin "G1"
+		)
+		(pin "2"
+		)
+		(pin "3"
+		)
+		(instances
+			(project ""
+				(path "/9ed354c1-be1e-4ed3-9daf-708fd38c762e"
+					(reference "J7")
 					(unit 1)
 				)
@@
 	)
 	(symbol
-		(lib_id "DB:SM04B-SRSS-TB")
-		(at 223.52 50.8 0)
-		(unit 1)
-		(exclude_from_sim yes)
-		(in_bom yes)
-		(on_board yes)
-		(dnp no)
-		(fields_autoplaced yes)
-		(property "Reference" "CN1"
-			(at 224.79 38.1 0)
-			(effects
-				(font
-					(size 1.27 1.27)
-				)
-			)
-		)
-		(property "Value" "SM04B-SRSS-TB"
-			(at 224.79 40.64 0)
-			(effects
-				(font
-					(size 1.27 1.27)
-				)
-			)
-		)
-		(property "Footprint" "footprints:JST_SH_SM04B-SRSS-TB"
-			(at 223.52 50.8 0)
-			(effects
-				(font
-					(size 1.27 1.27)
-				)
-				(hide yes)
-			)
-		)
-		(property "Datasheet" "http://parts.djgood.ca/en/part/24/info"
-			(at 223.52 50.8 0)
-			(effects
-				(font
-					(size 1.27 1.27)
-				)
-				(hide yes)
-			)
-		)
-		(property "Description" "Connector Header Surface Mount, Right Angle 4 position 0.039\" (1.00mm)"
-			(at 223.52 50.8 0)
-			(effects
-				(font
-					(size 1.27 1.27)
-				)
-				(hide yes)
-			)
-		)
-		(property "Category" "Connectors/Rectangular Connectors/Male Pins"
-			(at 223.52 50.8 0)
-			(effects
-				(font
-					(size 1.27 1.27)
-				)
-				(hide yes)
-			)
-		)
-		(property "MPN" "SM04B-SRSS-TB"
-			(at 223.52 50.8 0)
-			(effects
-				(font
-					(size 1.27 1.27)
-				)
-				(hide yes)
-			)
-		)
-		(property "Manufacturer" "JST Sales America Inc."
-			(at 223.52 50.8 0)
-			(effects
-				(font
-					(size 1.27 1.27)
-				)
-				(hide yes)
-			)
-		)
-		(property "Manufacturing Status" "Active"
-			(at 223.52 50.8 0)
-			(effects
-				(font
-					(size 1.27 1.27)
-				)
-				(hide yes)
-			)
-		)
-		(property "Part-DB ID" "24"
-			(at 223.52 50.8 0)
-			(effects
-				(font
-					(size 1.27 1.27)
-				)
-				(hide yes)
-			)
-		)
-		(pin "G2"
-		)
-		(pin "2"
-		)
-		(pin "G1"
-		)
-		(pin "1"
-		)
-		(pin "4"
-		)
-		(pin "3"
-		)
-		(instances
-			(project ""
-				(path "/9ed354c1-be1e-4ed3-9daf-708fd38c762e"
-					(reference "CN1")
-					(unit 1)
-				)
-			)
-		)
-	)
-	(symbol
 		(lib_id "power:GND")
 		(at 83.82 101.6 0)
@@
 	)
 	(sheet
-		(at 199.39 69.85)
+		(at 200.66 69.85)
 		(size 33.02 16.51)
 		(fields_autoplaced yes)
@@
 		)
 		(property "Sheetname" "nRF9151 - Power + RF"
-			(at 199.39 69.1384 0)
+			(at 200.66 69.1384 0)
 			(effects
 				(font
@@
 		)
 		(property "Sheetfile" "nrf9151_power_rf.kicad_sch"
-			(at 199.39 86.9446 0)
+			(at 200.66 86.9446 0)
 			(effects
 				(font
@@
 		)
 		(pin "LNA_EN" input
-			(at 232.41 77.47 0)
+			(at 233.68 77.47 0)
 			(effects
 				(font
@@
 		)
 		(pin "PWR_3V3H" input
-			(at 199.39 77.47 180)
-			(effects
-				(font
+			(at 200.66 77.47 180)
+			(effects
+				(font

Commit message: Publish PCB and Schematics
Parts:
- removed J4, J5: AA-CONTACT-SMD, footprints:AA-CONTACT-SMD, symbol DB:AA-CONTACT-SMD
- added J1, J2: KEYSTONE_254, footprints:KEYSTONE_254, symbol DB:KEYSTONE_254
- added J16: S2B-PH-SM4-TB, footprints:JST_PH_S2B-PH-SM4-TB_1x02-1MP_P2.00mm_Horizontal, symbol DB:S2B-PH-SM4-TB
- added J4, J5, J6, J7, J8, J9: 10129380-902001BLF, footprints:PinHeader_1x02_P2.54mm_Vertical_SMD_Pin1Left, symbol DB:10129380-902001BLF
- added JMP1, JMP2, JMP3, JMP4, JMP5, JMP6: QPC02SXGN-RC, symbol DB:QPC02SXGN-RC
- added TP1, TP2, TP3, TP4, TP5, TP6: RCWCTE, footprints:KOA_TEST_POINT_1206, symbol DB:RCWCTE
- J10: renamed from J7; footprint footprints:BM04B-SRSS-TB -> footprints:JST_SH_BM04B-SRSS-TB
- J3: footprint footprints:54-00125 -> footprints:TENSILITY_54-00125
Connections:
- net GND: now also J3.B, J16.G1, J16.G2, TP5.1, TP6.1; no longer J3.2
- net PANEL_DETECT: now also J3.C; no longer J3.3
- net I2C_SBUS_SCL renamed I2C_SBUS.SCL
- net I2C_SBUS_SDA renamed I2C_SBUS.SDA
- net Power Management/PWR_3V3_LS renamed PWR_3V3_LS_OUT
- net PWR_3V3_LS_OUT: now also J8.1 (Pin_1)
- removed net Power Management/PWR_SOLAR: J3.1
- new net BAT_N: J16.1 (NEG), J2.1
- new net BAT_P: J1.1, J16.2 (POS)
- new net PWR_3V3: J7.2 (Pin_2), J9.2 (Pin_2), TP4.1
- new net PWR_3V3_LS: J8.2 (Pin_2)
- new net PWR_BATT: J4.1 (Pin_1)
- new net PWR_BAT_IN: J4.2 (Pin_2), TP1.1
- new net PWR_PANEL: J5.1 (Pin_1)
- new net PWR_PANEL_IN: J3.A, J5.2 (Pin_2), TP2.1
- new net PWR_USB: J6.1 (Pin_1)
- new net PWR_USB_IN: J6.2 (Pin_2), TP3.1
- new net PWR_nRF52: J7.1 (Pin_1)
- new net PWR_nRF91: J9.1 (Pin_1)
Other:
- added sheet Battery Protection (battery-protection.kicad_sch)
- added sheet nRF52833 (nrf52833.kicad_sch)
- sheet Power Management ports: added I2C_PMIC{I2C}, PWR_3V3; removed I2C_PMIC, PWR_3V3H, STAT, nQON
- sheet USB ports: added PWR_USB_5V0, USB_D_N, USB_D_P; removed PWR_5V0_USB, USB_UART
- sheet nRF9151 - GPIO + UICC ports: added BLE_SPI{SPI}, I2C_PMIC{I2C}, I2C_SBUS{I2C}, UART0{UART}, UART1{UART}, nRF52_nRESET, nRF91_SWD{SWD}, {GPIO_BUS}; removed I2C_PMIC, I2C_SBUS, STAT, USB_UART, nQON
- note added: "Pair of SMD contacts form a 18650 cell holder"
- note added: "Power Test Points"
- note added: "Signal Test Points"
- note added: "to External Battery Pack (optional)"
- note removed: "Pair of SMD contacts form a 14430 cell holder"
- moved on the sheet: J10, J3
