File: usb_conn.kicad_sch (KiCad schematic)
At the start: 16 parts, among them CN2 USB4105-GF-A, U5 EXC-34CE121U, U8 USBLC6-4SC6, U9 FT234XD

Commit message: Add files via upload
Other:
- title: (none) -> USB Interface
Changed lines of the file:
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@@
 	(paper "A4")
 	(title_block
+		(title "USB Interface")
 		(date "2025-01-04")
 	)

Commit message: Publish PCB and Schematics
Parts:
- removed C28, C30: 0.1u 16V, footprints:C_0201_0603Metric, symbol DB:GRM033Z71C104KE14J
- removed C29: 10n, footprints:C_0402_1005Metric, symbol DB:CC0402KRX7R8BB103
- removed R21: 10K, footprints:R_0402_1005Metric, symbol DB:ERJ-2RKF1002X
- removed U9: FT234XD, footprints:FT234XD, symbol DB:FT234XD
- C42: renamed from C26; value 4.7u 10V -> 4u7 10V
- C43: renamed from C27; value 0.1u 16V -> 100n 16V; footprint footprints:C_0201_0603Metric -> footprints:C_0402_1005Metric; symbol DB:GRM033Z71C104KE14J -> DB:GRM155R71H104KE14D; Category Capacitors -> Capacitors/Ceramic Capacitors; MPN GRM033Z71C104KE14J -> GRM155R71H104KE14D; Part-DB ID 34 -> 132
- CN1: renamed from CN2; footprint footprints:GCT_USB4105-GF-A -> footprints:GCT_USB4105-XX
- U8: renamed from U5; footprint footprints:Panasonic_EXC34CE -> footprints:PANASONIC_EXCX4CE; now left out of the parts list
- U9: renamed from U8; footprint (none) -> footprints:ST_SOT-23-6; Category Circuit Protection/TVS Diodes -> Diodes/TVS
- renumbered C16 to C41, L3 to L5, R16 to R31, R17 to R32, R14 to R33, R15 to R34
Connections:
- net PWR_5V0_USB_IN is gone; now on net PWR_USB_5V0_IN: C41.1, CN1.A4 (VBUS), CN1.A9 (VBUS), CN1.B4 (VBUS), CN1.B9 (VBUS), L5.1
- net USB_CC1: no longer U9.1 (I/O1)
- net USB_CC2: no longer U9.3 (I/O2)
- net USB_CMC_D_P: now also U8.2; no longer U8.4
- net USB_D_N: now also U8.4; no longer U8.2
- net 5V0_USB renamed PWR_USB_5V0_IN
- no-connect marks 3 -> 4
Other:
- moved on the sheet: C41, C42, C43, CN1, L5, R31, R32, R33, R34, U8, U9
